File: Hardware/oscar_panel.kicad_pcb (KiCad board)
At the start: 2 copper layers, 71 x 128.5 mm, 15 parts

Commit message: Relocated and reorganised repository
Parts:
- removed the Ref** at (186.0, 151.0)
- added Ref**: Subminiature_Switch, Custom_Footprints:Sub_Miniature_Switch_MountingHole_3.5mm, F.Cu at (186.0, 151.0)
Other:
- board text added: "OSCAR Panel v2"
- board text removed: "OSCAR Panel v1"
Changed lines of the file:
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@@
   (page A4)
   (layers
-    (0 F.Cu signal hide)
-    (31 B.Cu signal)
+    (0 F.Cu signal)
+    (31 B.Cu signal hide)
     (34 B.Paste user)
     (35 F.Paste user)
@@
     (uvia_dia 0.3)
     (uvia_drill 0.1)
+  )
+  (module Custom_Footprints:Sub_Miniature_Switch_MountingHole_3.5mm (layer F.Cu)
+    (at 186 151)
+    (descr "Mounting Hole 6mm, no annular")
+    (tags "mounting hole 6mm no annular")
+    (fp_text reference Ref** (at 0 -5.4) (layer F.SilkS) hide
+      (effects (font (size 1 1) (thickness 0.15)))
+    )
+    (fp_text value Subminiature_Switch (at 0 5.1) (layer F.Fab) hide
+      (effects (font (size 1 1) (thickness 0.15)))
+    )
+    (fp_circle (center 0 0) (end 1.5 0) (layer Cmts.User) (width 0.15))
+    (fp_circle (center 0 0) (end 1.6 0) (layer F.CrtYd) (width 0.05))
+    (pad "" np_thru_hole circle (at 0 0) (size 3.5 3.5) (drill 3.5) (layers *.Cu *.Mask))
   )
   (module oscar_logo:oscar_logo (layer F.Cu)
@@
     (pad "" np_thru_hole circle (at 0 0) (size 7 7) (drill 7) (layers *.Cu *.Mask))
   )
-  (module Custom_Footprints:Sub_Miniature_Switch_MountingHole_3mm (layer F.Cu)
-    (at 186 151)
-    (descr "Mounting Hole 6mm, no annular")
-    (tags "mounting hole 6mm no annular")
-    (fp_text reference Ref** (at 0 -5.4) (layer F.SilkS) hide
-      (effects (font (size 1 1) (thickness 0.15)))
-    )
-    (fp_text value Subminiature_Switch (at 0 5.1) (layer F.Fab) hide
-      (effects (font (size 1 1) (thickness 0.15)))
-    )
-    (fp_circle (center 0 0) (end 1.5 0) (layer Cmts.User) (width 0.15))
-    (fp_circle (center 0 0) (end 1.6 0) (layer F.CrtYd) (width 0.05))
-    (pad "" np_thru_hole circle (at 0 0) (size 3 3) (drill 3) (layers *.Cu *.Mask))
-  )
   (module Custom_Footprints:Thonkiconn_Socket_MountingHole_6mm (layer F.Cu)
     (at 165 151)
@@
     (pad "" np_thru_hole circle (at 0 0) (size 6 6) (drill 6) (layers *.Cu *.Mask))
   )
-  (gr_text "OSCAR Panel v1" (at 159.8 44.1) (layer B.SilkS)
+  (gr_text "OSCAR Panel v2" (at 159.8 44.1) (layer B.SilkS)
     (effects (font (size 1 1) (thickness 0.15)) (justify mirror))
   )
